Commit message: added description package

File: src/racecar_description/urdf/racecar.xacro (robot description, xacro)
@@ -2,5 +2,5 @@
 <robot name="virtual_robot" xmlns:xacro="http://www.ros.org/wiki/xacro">
   <!-- Global namespace -->
-  <xacro:arg name="robot_name" default="car_1" />
+  <xacro:arg name="robot_name" default="" />
   <xacro:arg name="robot_skin" default="Blue" />
   <!-- inertial parameter macros -->
@@ -44,5 +44,5 @@
     <origin xyz="0.46 -0.135 -0.180" rpy="1.57 0 3.14" />
     <geometry>
-      <mesh filename="package://racecar_description/urdf/meshes/chassis.stl" scale="0.000990 0.0009375 0.0009375"/>
+      <mesh filename="package://racecar_description/meshes/chassis.stl" scale="0.000990 0.0009375 0.0009375"/>
     </geometry>
   </xacro:macro>
@@ -50,5 +50,5 @@
     <origin xyz="0 0 0" rpy="0 0 0" />
     <geometry>
-      <mesh filename="package://racecar_description/urdf/meshes/left_wheel.stl" />
+      <mesh filename="package://racecar_description/meshes/left_wheel.stl" />
     </geometry>
   </xacro:macro>
@@ -56,5 +56,5 @@
     <origin xyz="0 0 0" rpy="0 0 0" />
     <geometry>
-      <mesh filename="package://racecar_description/urdf/meshes/right_wheel.stl" />
+      <mesh filename="package://racecar_description/meshes/right_wheel.stl" />
     </geometry>
   </xacro:macro>
@@ -62,5 +62,5 @@
     <origin xyz="0 0 0" rpy="0 0 0" />
     <geometry>
-      <mesh filename="package://racecar_description/urdf/meshes/left_wheel.stl" />
+      <mesh filename="package://racecar_description/meshes/left_wheel.stl" />
     </geometry>
   </xacro:macro>
@@ -68,5 +68,5 @@
     <origin xyz="0 0 0" rpy="0 0 0" />
     <geometry>
-      <mesh filename="package://racecar_description/urdf/meshes/right_wheel.stl" />
+      <mesh filename="package://racecar_description/meshes/right_wheel.stl" />
     </geometry>
   </xacro:macro>
@@ -74,5 +74,5 @@
     <origin xyz="0 0 0" rpy="0 0 0" />
     <geometry>
-      <mesh filename="package://racecar_description/urdf/meshes/hinge.stl" />
+      <mesh filename="package://racecar_description/meshes/hinge.stl" />
     </geometry>
   </xacro:macro>
@@ -80,5 +80,5 @@
     <origin xyz="0 0 0" rpy="0 0 0" />
     <geometry>
-      <mesh filename="package://racecar_description/urdf/meshes/hinge.stl" />
+      <mesh filename="package://racecar_description/meshes/hinge.stl" />
     </geometry>
   </xacro:macro>
@@ -121,6 +121,6 @@
   </xacro:macro>
   <!-- Add chassis and it's inertia link -->
-  <link name="$(arg robot_name)_base_link"/>
-  <link name="$(arg robot_name)_chassis">
+  <link name="$(arg robot_name)base_link"/>
+  <link name="$(arg robot_name)chassis">
     <visual>
       <xacro:chassis_geometry/>
@@ -128,21 +128,21 @@
     </visual>
   </link>
-  <joint name="$(arg robot_name)_base_link_joint" type="fixed">
+  <joint name="$(arg robot_name)base_link_joint" type="fixed">
     <origin xyz="0 0 0.05" rpy="0 0 0" />
-    <parent link="$(arg robot_name)_base_link" />
-    <child link="$(arg robot_name)_chassis" />
-  </joint>
-  <link name="$(arg robot_name)_chassis_inertia">
+    <parent link="$(arg robot_name)base_link" />
+    <child link="$(arg robot_name)chassis" />
+  </joint>
+  <link name="$(arg robot_name)chassis_inertia">
     <inertial>
       <xacro:chassis_inertial_params />
     </inertial>
   </link>
-  <joint name="$(arg robot_name)_chassis_inertia_joint" type="fixed">
-    <origin xyz="0 0 0" rpy="0 0 0" />
-    <parent link="$(arg robot_name)_chassis" />
-    <child link="$(arg robot_name)_chassis_inertia" />
+  <joint name="$(arg robot_name)chassis_inertia_joint" type="fixed">
+    <origin xyz="0 0 0" rpy="0 0 0" />
+    <parent link="$(arg robot_name)chassis" />
+    <child link="$(arg robot_name)chassis_inertia" />
   </joint>
   <!-- Add the left rear wheel with its joints and tranmissions -->
-  <link name="$(arg robot_name)_left_rear_wheel">
+  <link name="$(arg robot_name)left_rear_wheel">
     <inertial>
       <xacro:left_wheels_inertial_params />
@@ -156,14 +156,14 @@
     </collision>
   </link>
-  <joint name="$(arg robot_name)_left_rear_wheel_joint" type="continuous">
+  <joint name="$(arg robot_name)left_rear_wheel_joint" type="continuous">
     <origin xyz="0 0.1 0" rpy="1.5708 0 0" />
-    <parent link="$(arg robot_name)_chassis" />
-    <child link="$(arg robot_name)_left_rear_wheel" />
+    <parent link="$(arg robot_name)chassis" />
+    <child link="$(arg robot_name)left_rear_wheel" />
     <axis xyz="0 0 -1" />
     <limit effort="10" velocity="100" />
   </joint>
-  <xacro:wheel_transmission name="$(arg robot_name)_left_rear_wheel" />
+  <xacro:wheel_transmission name="$(arg robot_name)left_rear_wheel" />
   <!-- Add the right rear wheel with its joints and tranmissions -->
-  <link name="$(arg robot_name)_right_rear_wheel">
+  <link name="$(arg robot_name)right_rear_wheel">
     <inertial>
       <xacro:right_wheels_inertial_params />
@@ -177,14 +177,14 @@
     </collision>
   </link>
-  <joint name="$(arg robot_name)_right_rear_wheel_joint" type="continuous">
+  <joint name="$(arg robot_name)right_rear_wheel_joint" type="continuous">
     <origin xyz="0 -0.1 0" rpy="1.5708 0 0" />
-    <parent link="$(arg robot_name)_chassis" />
-    <child link="$(arg robot_name)_right_rear_wheel" />
+    <parent link="$(arg robot_name)chassis" />
+    <child link="$(arg robot_name)right_rear_wheel" />
     <axis xyz="0 0 -1" />
     <limit effort="10" velocity="100" />
   </joint>
-  <xacro:wheel_transmission name="$(arg robot_name)_right_rear_wheel" />
+  <xacro:wheel_transmission name="$(arg robot_name)right_rear_wheel" />
   <!-- Add the left steering hinge with its joints and tranmissions -->
-  <link name="$(arg robot_name)_left_steering_hinge">
+  <link name="$(arg robot_name)left_steering_hinge">
     <inertial>
       <xacro:steering_hinge_inertial_params />
@@ -195,14 +195,14 @@
     </visual>
   </link>
-  <joint name="$(arg robot_name)_left_steering_hinge_joint" type="revolute">
+  <joint name="$(arg robot_name)left_steering_hinge_joint" type="revolute">
     <origin xyz="0.325 0.1 0" rpy="0 1.5708 0" />
-    <parent link="$(arg robot_name)_chassis" />
-    <child link="$(arg robot_name)_left_steering_hinge" />
+    <parent link="$(arg robot_name)chassis" />
+    <child link="$(arg robot_name)left_steering_hinge" />
     <axis xyz="-1 0 0" />
     <limit lower="-1.0" upper="1.0" effort="10" velocity="100" />
   </joint>
-  <xacro:steering_hinge_transmission name="$(arg robot_name)_left_steering_hinge" />
+  <xacro:steering_hinge_transmission name="$(arg robot_name)left_steering_hinge" />
   <!-- Add the right steering hinge with its joints and tranmissions -->
-  <link name="$(arg robot_name)_right_steering_hinge">
+  <link name="$(arg robot_name)right_steering_hinge">
     <inertial>
       <xacro:steering_hinge_inertial_params />
@@ -213,14 +213,14 @@
     </visual>
   </link>
-  <joint name="$(arg robot_name)_right_steering_hinge_joint" type="continuous">
+  <joint name="$(arg robot_name)right_steering_hinge_joint" type="revolute">
     <origin xyz="0.325 -0.1 0" rpy="0 1.5708 0" />
-    <parent link="$(arg robot_name)_chassis" />
-    <child link="$(arg robot_name)_right_steering_hinge" />
+    <parent link="$(arg robot_name)chassis" />
+    <child link="$(arg robot_name)right_steering_hinge" />
     <axis xyz="-1 0 0" />
     <limit lower="-1.0" upper="1.0" effort="10" velocity="100" />
   </joint>
-  <xacro:steering_hinge_transmission name="$(arg robot_name)_right_steering_hinge" />
+  <xacro:steering_hinge_transmission name="$(arg robot_name)right_steering_hinge" />
   <!-- Add the left front wheel with its joints and tranmissions -->
-  <link name="$(arg robot_name)_left_front_wheel">
+  <link name="$(arg robot_name)left_front_wheel">
     <inertial>
       <xacro:left_wheels_inertial_params />
@@ -234,14 +234,14 @@
     </collision>
   </link>
-  <joint name="$(arg robot_name)_left_front_wheel_joint" type="continuous">
+  <joint name="$(arg robot_name)left_front_wheel_joint" type="continuous">
     <origin xyz="0 0 0" rpy="1.5708 0 0" />
-    <parent link="$(arg robot_name)_left_steering_hinge" />
-    <child link="$(arg robot_name)_left_front_wheel" />
+    <parent link="$(arg robot_name)left_steering_hinge" />
+    <child link="$(arg robot_name)left_front_wheel" />
     <axis xyz="0 0 -1" />
     <limit effort="10" velocity="100" />
   </joint>
-  <xacro:wheel_transmission name="$(arg robot_name)_left_front_wheel" />
+  <xacro:wheel_transmission name="$(arg robot_name)left_front_wheel" />
   <!-- Add the left front wheel with its joints and tranmissions -->
-  <link name="$(arg robot_name)_right_front_wheel">
+  <link name="$(arg robot_name)right_front_wheel">
     <inertial>
       <xacro:right_wheels_inertial_params />
@@ -255,14 +255,14 @@
     </collision>
   </link>
-  <joint name="$(arg robot_name)_right_front_wheel_joint" type="continuous">
+  <joint name="$(arg robot_name)right_front_wheel_joint" type="continuous">
     <origin xyz="0 0 0" rpy="1.5708 0 0" />
-    <parent link="$(arg robot_name)_right_steering_hinge" />
-    <child link="$(arg robot_name)_right_front_wheel" />
+    <parent link="$(arg robot_name)right_steering_hinge" />
+    <child link="$(arg robot_name)right_front_wheel" />
     <axis xyz="0 0 -1" />
     <limit effort="10" velocity="100"/>
   </joint>
-  <xacro:wheel_transmission name="$(arg robot_name)_right_front_wheel" />
+  <xacro:wheel_transmission name="$(arg robot_name)right_front_wheel" />
   <!-- Add Hokuyo laser scanner -->
-  <link name="$(arg robot_name)_laser">
+  <link name="$(arg robot_name)laser">
     <inertial>
       <xacro:hokuyo_inertial_params />
@@ -277,17 +277,17 @@
       <origin xyz="0 0 0" rpy="0 0 0"/>
       <geometry>
-        <mesh filename="package://racecar_description/urdf/meshes/hokuyo.stl"/>
+        <mesh filename="package://racecar_description/meshes/hokuyo.stl"/>
         <material name="grey" />
       </geometry>
     </visual>
   </link>
-  <joint name="$(arg robot_name)_hokuyo_joint" type="fixed">
+  <joint name="$(arg robot_name)hokuyo_joint" type="fixed">
     <origin xyz="0.125 0.0 0.155" rpy="0 0 0"/>
-    <parent link="$(arg robot_name)_chassis" />
-    <child link="$(arg robot_name)_laser" />
+    <parent link="$(arg robot_name)chassis" />
+    <child link="$(arg robot_name)laser" />
     <axis xyz="0 0 1" />
   </joint>
   <!-- camera class (spawn parameters) -->
-  <link name="$(arg robot_name)_link">
+  <link name="$(arg robot_name)link">
     <inertial>
       <mass value="1e-5" />
@@ -309,40 +309,27 @@
     </visual>
   </link>
-  <joint name="$(arg robot_name)_joint" type="fixed">
+  <joint name="$(arg robot_name)joint" type="fixed">
     <origin xyz="0.390 0 0.025" rpy="0 0 0"/>
-    <parent link="$(arg robot_name)_chassis"/>
-    <child link="$(arg robot_name)_link"/>
+    <parent link="$(arg robot_name)chassis"/>
+    <child link="$(arg robot_name)link"/>
     <axis xyz="0 0 1" />
     <!-- <limit lower="0.0" upper="0.0" effort="0.0" velocity="0.0" /> -->
   </joint>
   <!-- camera lenses -->
-  <link name="$(arg robot_name)_camera_link">
+  <link name="$(arg robot_name)right_link">
     <inertial>
       <mass value="1e-5" />
-      <origin xyz="-0.25 0 0.025" rpy="0 0 0"/>
+      <origin xyz="-2.5 0 1.75" rpy="0 .57 0"/>
       <inertia ixx="1e-6" ixy="0" ixz="0" iyy="1e-6" iyz="0" izz="1e-6" />
     </inertial>
   </link>
-  <link name="$(arg robot_name)_right_link">
-    <inertial>
-      <mass value="1e-5" />
-      <origin xyz="0 0 0.025" rpy="0 0 0"/>
-      <inertia ixx="1e-6" ixy="0" ixz="0" iyy="1e-6" iyz="0" izz="1e-6" />
-    </inertial>
-  </link>
-  <joint name="$(arg robot_name)_left_joint" type="fixed">
-    <origin xyz="0 0 0.035" rpy="0 0 0"/>
-    <parent link="$(arg robot_name)_link"/>
-    <child link="$(arg robot_name)_camera_link"/>
+  <joint name="$(arg robot_name)right_joint" type="fixed">
+    <origin xyz="0 -0.06 0.025" rpy="0 0 0"/>
+    <parent link="$(arg robot_name)link"/>
+    <child link="$(arg robot_name)right_link"/>
     <axis xyz="0 0 1" />
   </joint>
-  <joint name="$(arg robot_name)_right_joint" type="fixed">
-    <origin xyz="0 -0.06 0.025" rpy="0 0 0"/>
-    <parent link="$(arg robot_name)_link"/>
-    <child link="$(arg robot_name)_right_link"/>
-    <axis xyz="0 0 1" />
-  </joint>
   <!-- Gazebo references -->
-  <gazebo reference="$(arg robot_name)_chassis">
+  <gazebo reference="$(arg robot_name)chassis">
     <mu1 value="0.0"/>
     <mu2 value="0.0"/>
@@ -351,5 +338,5 @@
     <material>Gazebo/$(arg robot_skin)</material>
   </gazebo>
-  <gazebo reference="$(arg robot_name)_left_rear_wheel">
+  <gazebo reference="$(arg robot_name)left_rear_wheel">
     <mu1 value="1.0"/>
     <mu2 value="1.0"/>
@@ -359,5 +346,5 @@
     <material>Gazebo/Black</material>
   </gazebo>
-  <gazebo reference="$(arg robot_name)_right_rear_wheel">
+  <gazebo reference="$(arg robot_name)right_rear_wheel">
     <mu1 value="1.0"/>
     <mu2 value="1.0"/>
@@ -367,5 +354,5 @@
     <material>Gazebo/Black</material>
   </gazebo>
-  <gazebo reference="$(arg robot_name)_left_front_wheel">
+  <gazebo reference="$(arg robot_name)left_front_wheel">
     <mu1 value="1.0"/>
     <mu2 value="1.0"/>
@@ -375,5 +362,5 @@
     <material>Gazebo/Black</material>
   </gazebo>
-  <gazebo reference="$(arg robot_name)_right_front_wheel">
+  <gazebo reference="$(arg robot_name)right_front_wheel">
     <mu1 value="1.0"/>
     <mu2 value="1.0"/>
@@ -383,5 +370,5 @@
     <material>Gazebo/Black</material>
   </gazebo>
-  <!-- Gazebo plugins -->
+  <!-- Gazebo plugins
   <gazebo>
     <plugin name="gazebo_ros_control" filename="libgazebo_ros_control.so">
@@ -389,11 +376,11 @@
       <robotSimType>gazebo_ros_control/DefaultRobotHWSim</robotSimType>
     </plugin>
-  </gazebo>
-  <!-- Odometry (cheap hack) -->
+  </gazebo>-->
+  <!-- Odometry (cheap hack)
   <gazebo>
     <plugin name="p3d_base_controller" filename="libgazebo_ros_p3d.so">
       <alwaysOn>true</alwaysOn>
       <updateRate>50.0</updateRate>
-      <bodyName>$(arg robot_name)_base_link</bodyName>
+      <bodyName>$(arg robot_name)base_link</bodyName>
       <topicName>/$(arg robot_name)/ground_truth</topicName>
       <gaussianNoise>0.01</gaussianNoise>
@@ -402,78 +389,43 @@
       <rpyOffsets>0 0 0</rpyOffsets>
     </plugin>
-  </gazebo>
+  </gazebo> -->
     <!-- hokuyo -->
   <xacro:unless value="$(optenv DISABLE_GAZEBO_LASER false)">
-    <gazebo reference="$(arg robot_name)_laser">
-      <material>Gazebo/Grey</material>
-      <sensor type="ray" name="$(arg robot_name)_hokuyo_sensor">
-        <pose>0 0 0.0124 0 0 0</pose>
-        <visualize>false</visualize>
-        <update_rate>40</update_rate>
-        <ray>
-          <scan>
-            <horizontal>
-              <samples>1081</samples>
-              <resolution>1</resolution>
-              <min_angle>-2.3561944902</min_angle>
-              <max_angle>2.3561944902</max_angle>
-            </horizontal>
-          </scan>
-          <range>
-            <min>0.1</min>
-            <max>30.0</max>
-            <resolution>0.01</resolution>
-          </range>
-          <noise>
-            <mean>0.0</mean>
-            <stddev>0.01</stddev>
-          </noise>
-        </ray>
-        <plugin name="gazebo_ros_hokuyo_controller" filename="libgazebo_ros_laser.so">
-          <topicName>/$(arg robot_name)/scan</topicName>
-          <frameName>$(arg robot_name)_laser</frameName>
-        </plugin>
-      </sensor>
-    </gazebo>
-  </xacro:unless>
-  <!-- camera object -->
-  <xacro:unless value="$(optenv DISABLE_GAZEBO_CAMERA false)">
-    <gazebo reference="$(arg robot_name)_camera_link">
-      <sensor type="camera" name="$(arg robot_name)_left_sensor">
-        <update_rate>30.0</update_rate>
-        <!-- math.atan(320 / 687.8065795898438) * 2 -->
-        <camera name="front_camera">
-          <!-- horizontal_fov>0.8709216071359963</horizontal_fov -->
-          <horizontal_fov>1.74</horizontal_fov>
-          <image>
-            <width>1920</width>
-            <height>1080</height>
-            <format>B8G8R8</format>
-          </image>
-          <clip>
-            <near>0.02</near>
-            <far>300</far>
-          </clip>
-          <noise>
-            <type>gaussian</type>
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