Commit message: fixed urdf file

File: src/racecar_description/urdf/racecar.urdf.xacro (robot description, xacro)
@@ -1,4 +1,4 @@
 <?xml version="1.0"?>
-<robot name="virtual_robot" xmlns:xacro="http://www.ros.org/wiki/xacro">
+<robot name="racecar" xmlns:xacro="http://www.ros.org/wiki/xacro">
   <!-- Global namespace -->
   <xacro:arg name="robot_name" default="" />
@@ -288,5 +288,4 @@
     <axis xyz="0 0 1" />
   </joint>
-  <!-- camera class (spawn parameters) -->
   <link name="$(arg robot_name)link">
     <inertial>
@@ -316,5 +315,4 @@
     <!-- <limit lower="0.0" upper="0.0" effort="0.0" velocity="0.0" /> -->
   </joint>
-  <!-- camera lenses -->
   <link name="$(arg robot_name)right_link">
     <inertial>
@@ -370,5 +368,5 @@
     <material>Gazebo/Black</material>
   </gazebo>
-  <!-- Gazebo plugins
+  <!-- Gazebo plugins -->
   <gazebo>
     <plugin name="gazebo_ros_control" filename="libgazebo_ros_control.so">
@@ -376,6 +374,6 @@
       <robotSimType>gazebo_ros_control/DefaultRobotHWSim</robotSimType>
     </plugin>
-  </gazebo>-->
-  <!-- Odometry (cheap hack)
+  </gazebo>
+  <!-- Odometry (cheap hack) -->
   <gazebo>
     <plugin name="p3d_base_controller" filename="libgazebo_ros_p3d.so">
@@ -389,43 +387,37 @@
       <rpyOffsets>0 0 0</rpyOffsets>
     </plugin>
-  </gazebo> -->
+  </gazebo>
     <!-- hokuyo -->
   <xacro:unless value="$(optenv DISABLE_GAZEBO_LASER false)">
     <gazebo reference="$(arg robot_name)laser">
-      <sensor type="gpu_ray" name="head_hokuyo_sensor">
-    <ray>
-      <scan>
-        <horizontal>
-          <samples>720</samples>
-          <resolution>1</resolution>
-          <min_angle>-1.570796</min_angle>
-          <max_angle>1.570796</max_angle>
-        </horizontal>
-      </scan>
-      <range>
-        <min>0.10</min>
-        <max>30.0</max>
-        <resolution>0.01</resolution>
-      </range>
-      <!-- Using gazebo's noise instead of plugin's -->
-      <noise>
-        <type>gaussian</type>
-        <mean>0.0</mean>
-        <stddev>0.01</stddev>
-      </noise>
-    </ray>
-    <!-- Using gazebo's update rate instead of plugin's -->
-    <update_rate>30</update_rate>
-    <plugin name="gazebo_ros_head_hokuyo_controller" filename="libgazebo_ros_ray_sensor.so">
-      <!-- Change namespace and output topic so published topic is /rrbot/laser/scan -->
-      <ros>
-        <namespace>/rrbot/laser</namespace>
-        <argument>~/out:=scan</argument>
-      </ros>
-      <!-- Set output to sensor_msgs/LaserScan to get same output type as gazebo_ros_laser -->
-      <output_type>sensor_msgs/LaserScan</output_type>
-      <!-- <frame_name> ommited, will default to hokuo_link -->
-    </plugin>
-  </sensor>
+      <material>Gazebo/Grey</material>
+      <sensor type="ray" name="$(arg robot_name)hokuyo_sensor">
+        <pose>0 0 0.0124 0 0 0</pose>
+        <visualize>false</visualize>
+        <update_rate>40</update_rate>
+        <ray>
+          <scan>
+            <horizontal>
+              <samples>1081</samples>
+              <resolution>1</resolution>
+              <min_angle>-2.3561944902</min_angle>
+              <max_angle>2.3561944902</max_angle>
+            </horizontal>
+          </scan>
+          <range>
+            <min>0.1</min>
+            <max>30.0</max>
+            <resolution>0.01</resolution>
+          </range>
+          <noise>
+            <mean>0.0</mean>
+            <stddev>0.01</stddev>
+          </noise>
+        </ray>
+        <plugin name="hokuyo_controller" filename="libgazebo_ros_laser.so">
+          <topicName>/$(arg robot_name)/scan</topicName>
+          <frameName>$(arg robot_name)laser</frameName>
+        </plugin>
+      </sensor>
     </gazebo>
   </xacro:unless>

Commit message: added gazebo simulation

File: src/racecar_description/urdf/racecar.urdf.xacro (robot description, xacro)
@@ -44,5 +44,5 @@
     <origin xyz="0.46 -0.135 -0.180" rpy="1.57 0 3.14" />
     <geometry>
-      <mesh filename="package://racecar_description/meshes/chassis.stl" scale="0.000990 0.0009375 0.0009375"/>
+      <mesh filename="file://$(find racecar_description)/meshes/chassis.stl" scale="0.000990 0.0009375 0.0009375"/>
     </geometry>
   </xacro:macro>
@@ -50,5 +50,5 @@
     <origin xyz="0 0 0" rpy="0 0 0" />
     <geometry>
-      <mesh filename="package://racecar_description/meshes/left_wheel.stl" />
+      <mesh filename="file://$(find racecar_description)/meshes/left_wheel.stl" />
     </geometry>
   </xacro:macro>
@@ -56,5 +56,5 @@
     <origin xyz="0 0 0" rpy="0 0 0" />
     <geometry>
-      <mesh filename="package://racecar_description/meshes/right_wheel.stl" />
+      <mesh filename="file://$(find racecar_description)/meshes/right_wheel.stl" />
     </geometry>
   </xacro:macro>
@@ -62,5 +62,5 @@
     <origin xyz="0 0 0" rpy="0 0 0" />
     <geometry>
-      <mesh filename="package://racecar_description/meshes/left_wheel.stl" />
+      <mesh filename="file://$(find racecar_description)/meshes/left_wheel.stl" />
     </geometry>
   </xacro:macro>
@@ -68,5 +68,5 @@
     <origin xyz="0 0 0" rpy="0 0 0" />
     <geometry>
-      <mesh filename="package://racecar_description/meshes/right_wheel.stl" />
+      <mesh filename="file://$(find racecar_description)/meshes/right_wheel.stl" />
     </geometry>
   </xacro:macro>
@@ -74,5 +74,5 @@
     <origin xyz="0 0 0" rpy="0 0 0" />
     <geometry>
-      <mesh filename="package://racecar_description/meshes/hinge.stl" />
+      <mesh filename="file://$(find racecar_description)/meshes/hinge.stl" />
     </geometry>
   </xacro:macro>
@@ -80,5 +80,5 @@
     <origin xyz="0 0 0" rpy="0 0 0" />
     <geometry>
-      <mesh filename="package://racecar_description/meshes/hinge.stl" />
+      <mesh filename="file://$(find racecar_description)/meshes/hinge.stl" />
     </geometry>
   </xacro:macro>
@@ -277,5 +277,5 @@
       <origin xyz="0 0 0" rpy="0 0 0"/>
       <geometry>
-        <mesh filename="package://racecar_description/meshes/hokuyo.stl"/>
+        <mesh filename="file://$(find racecar_description)/meshes/hokuyo.stl"/>
         <material name="grey" />
       </geometry>
@@ -368,5 +368,5 @@
     <material>Gazebo/Black</material>
   </gazebo>
-  <!-- Gazebo plugins -->
+  <!-- Gazebo plugins
   <gazebo>
     <plugin name="gazebo_ros_control" filename="libgazebo_ros_control.so">
@@ -375,5 +375,4 @@
     </plugin>
   </gazebo>
-  <!-- Odometry (cheap hack) -->
   <gazebo>
     <plugin name="p3d_base_controller" filename="libgazebo_ros_p3d.so">
@@ -388,5 +387,4 @@
     </plugin>
   </gazebo>
-    <!-- hokuyo -->
   <xacro:unless value="$(optenv DISABLE_GAZEBO_LASER false)">
     <gazebo reference="$(arg robot_name)laser">
@@ -422,4 +420,5 @@
     </gazebo>
   </xacro:unless>
+-->
   <material name="black">
     <color rgba="0.0 0.0 0.0 1.0"/>

Commit message: fixed launch file

File: src/racecar_description/urdf/racecar.urdf.xacro (robot description, xacro)
@@ -152,5 +152,5 @@
       <material name="black" />
     </visual>
-    <collision>robot
+    <collision>
       <xacro:left_wheels_collision_geometry />
     </collision>

Commit message: fixed urdf file

File: src/racecar_description/urdf/racecar.urdf.xacro (robot description, xacro)
@@ -1,4 +1,5 @@
 <?xml version="1.0"?>
-<robot name="racecar" xmlns:xacro="http://www.ros.org/wiki/xacro">
+<robot name="racecar"
+  xmlns:xacro="http://www.ros.org/wiki/xacro">
   <!-- Global namespace -->
   <xacro:arg name="robot_name" default="" />
@@ -8,35 +9,25 @@
     <origin xyz="0.1477 0 0" rpy="0 0 0" />
     <mass value="4.0" />
-    <inertia ixx="0.010609" ixy="0"          ixz="0"
-                            iyy="0.050409"   iyz="0"
-                                             izz="0.05865" />
+    <inertia ixx="0.010609" ixy="0" ixz="0" iyy="0.050409" iyz="0" izz="0.05865" />
   </xacro:macro>
   <xacro:macro name="left_wheels_inertial_params">
     <origin xyz="0 0 -0.0225" rpy="0 0 0" />
     <mass value="0.34055" />
-    <inertia ixx="0.00026046" ixy="0"          ixz="0"
-                              iyy="0.00026046" iyz="0"
-                                               izz="0.00041226" />
+    <inertia ixx="0.00026046" ixy="0" ixz="0" iyy="0.00026046" iyz="0" izz="0.00041226" />
   </xacro:macro>
   <xacro:macro name="right_wheels_inertial_params">
     <origin xyz="0 0 0.0225" rpy="0 0 0" />
     <mass value="0.34055" />
-    <inertia ixx="0.00026046" ixy="0"          ixz="0"
-                              iyy="0.00026046" iyz="0"
-                                               izz="0.00041226" />
+    <inertia ixx="0.00026046" ixy="0" ixz="0" iyy="0.00026046" iyz="0" izz="0.00041226" />
   </xacro:macro>
   <xacro:macro name="steering_hinge_inertial_params">
     <origin xyz="0 0 0" rpy="0 0 0" />
     <mass value="0.100" />
-    <inertia ixx="4E-06" ixy="0"           ixz="0"
-                              iyy="4E-06"  iyz="0"
-                                                izz="4E-06" />
+    <inertia ixx="4E-06" ixy="0" ixz="0" iyy="4E-06" iyz="0" izz="4E-06" />
   </xacro:macro>
   <xacro:macro name="hokuyo_inertial_params">
     <origin xyz="0 0 0" rpy="0 0 0" />
     <mass value="0.130" />
-    <inertia ixx="4E-06" ixy="0"           ixz="0"
-                              iyy="4E-06"  iyz="0"
-                                                izz="4E-06" />
+    <inertia ixx="4E-06" ixy="0" ixz="0" iyy="4E-06" iyz="0" izz="4E-06" />
   </xacro:macro>
   <!-- geometry macros -->
@@ -264,5 +255,5 @@
   <xacro:wheel_transmission name="$(arg robot_name)right_front_wheel" />
   <!-- Add Hokuyo laser scanner -->
-  <link name="$(arg robot_name)laser">
+  <link name="$(arg robot_name)laser_link">
     <inertial>
       <xacro:hokuyo_inertial_params />
@@ -285,5 +276,5 @@
     <origin xyz="0.125 0.0 0.155" rpy="0 0 0"/>
     <parent link="$(arg robot_name)chassis" />
-    <child link="$(arg robot_name)laser" />
+    <child link="$(arg robot_name)laser_link" />
     <axis xyz="0 0 1" />
   </joint>
@@ -328,10 +319,24 @@
     <axis xyz="0 0 1" />
   </joint>
+  <ros2_control name="GazeboSystem" type="system">
+    <hardware>
+      <plugin>gazebo_ros2_control/GazeboSystem</plugin>
+    </hardware>
+    <joint name="slider_to_cart">
+      <command_interface name="effort">
+        <param name="min">-1000</param>
+        <param name="max">1000</param>
+      </command_interface>
+      <state_interface name="position"/>
+      <state_interface name="velocity"/>
+      <state_interface name="effort"/>
+    </joint>
+  </ros2_control>
   <!-- Gazebo references -->
   <gazebo reference="$(arg robot_name)chassis">
     <mu1 value="0.0"/>
     <mu2 value="0.0"/>
-    <kp  value="10000000.0" />
-    <kd  value="1.0" />
+    <kp value="10000000.0" />
+    <kd value="1.0" />
     <material>Gazebo/$(arg robot_skin)</material>
   </gazebo>
@@ -339,6 +344,6 @@
     <mu1 value="1.0"/>
     <mu2 value="1.0"/>
-    <kp  value="10000000.0" />
-    <kd  value="1.0" />
+    <kp value="10000000.0" />
+    <kd value="1.0" />
     <fdir1 value="1 0 0"/>
     <material>Gazebo/Black</material>
@@ -347,6 +352,6 @@
     <mu1 value="1.0"/>
     <mu2 value="1.0"/>
-    <kp  value="10000000.0" />
-    <kd  value="1.0" />
+    <kp value="10000000.0" />
+    <kd value="1.0" />
     <fdir1 value="1 0 0"/>
     <material>Gazebo/Black</material>
@@ -355,6 +360,6 @@
     <mu1 value="1.0"/>
     <mu2 value="1.0"/>
-    <kp  value="10000000.0" />
-    <kd  value="1.0" />
+    <kp value="10000000.0" />
+    <kd value="1.0" />
     <fdir1 value="0 0 1"/>
     <material>Gazebo/Black</material>
@@ -363,6 +368,6 @@
     <mu1 value="1.0"/>
     <mu2 value="1.0"/>
-    <kp  value="10000000.0" />
-    <kd  value="1.0" />
+    <kp value="10000000.0" />
+    <kd value="1.0" />
     <fdir1 value="0 0 1"/>
     <material>Gazebo/Black</material>
@@ -388,37 +393,40 @@
   </gazebo>
   <xacro:unless value="$(optenv DISABLE_GAZEBO_LASER false)">
-    <gazebo reference="$(arg robot_name)laser">
-      <material>Gazebo/Grey</material>
-      <sensor type="ray" name="$(arg robot_name)hokuyo_sensor">
-        <pose>0 0 0.0124 0 0 0</pose>
-        <visualize>false</visualize>
-        <update_rate>40</update_rate>
-        <ray>
-          <scan>
-            <horizontal>
-              <samples>1081</samples>
-              <resolution>1</resolution>
-              <min_angle>-2.3561944902</min_angle>
-              <max_angle>2.3561944902</max_angle>
-            </horizontal>
-          </scan>
-          <range>
-            <min>0.1</min>
-            <max>30.0</max>
-            <resolution>0.01</resolution>
-          </range>
-          <noise>
-            <mean>0.0</mean>
-            <stddev>0.01</stddev>
-          </noise>
-        </ray>
-        <plugin name="hokuyo_controller" filename="libgazebo_ros_laser.so">
-          <topicName>/$(arg robot_name)/scan</topicName>
-          <frameName>$(arg robot_name)laser</frameName>
-        </plugin>
-      </sensor>
-    </gazebo>
   </xacro:unless>
 -->
+  <gazebo reference="$(arg robot_name)laser_link">
+    <sensor name="$(arg robot_name)hokuyo_sensor" type="gpu_ray">
+      <visualize>true</visualize>
+      <update_rate>40</update_rate>
+      <pose>0 0 0.0124 0 0 0</pose>
+      <ray>
+        <scan>
+          <horizontal>
+            <samples>1081</samples>
+            <resolution>1</resolution>
+            <min_angle>-2.3561944902</min_angle>
+            <max_angle>2.3561944902</max_angle>
+          </horizontal>
+        </scan>
+        <range>
+          <min>0.1</min>
+          <max>30.0</max>
+          <resolution>0.01</resolution>
+        </range>
+        <noise>
+          <mean>0.0</mean>
+          <stddev>0.01</stddev>
+        </noise>
+      </ray>
+      <plugin name="scan" filename="libgazebo_ros_ray_sensor.so">
+        <ros>
+          <namespace>/$(arg robot_name)</namespace>
+          <remapping>~/out:=scan</remapping>
+        </ros>
+        <output_type>sensor_msgs/LaserScan</output_type>
+        <frame_name>$(arg robot_name)laser_link</frame_name>
+      </plugin>
+    </sensor>
+  </gazebo>
   <material name="black">
     <color rgba="0.0 0.0 0.0 1.0"/>

Commit message: got the ros2_control interface running

File: src/racecar_description/urdf/racecar.urdf.xacro (robot description, xacro)
@@ -35,5 +35,5 @@
     <origin xyz="0.46 -0.135 -0.180" rpy="1.57 0 3.14" />
     <geometry>
-      <mesh filename="file://$(find racecar_description)/meshes/chassis.stl" scale="0.000990 0.0009375 0.0009375"/>
+      <mesh filename="package://racecar_description/meshes/chassis.stl" scale="0.000990 0.0009375 0.0009375"/>
     </geometry>
   </xacro:macro>
@@ -41,5 +41,5 @@
     <origin xyz="0 0 0" rpy="0 0 0" />
     <geometry>
-      <mesh filename="file://$(find racecar_description)/meshes/left_wheel.stl" />
+      <mesh filename="package://racecar_description/meshes/left_wheel.stl" />
     </geometry>
   </xacro:macro>
@@ -47,5 +47,5 @@
     <origin xyz="0 0 0" rpy="0 0 0" />
     <geometry>
-      <mesh filename="file://$(find racecar_description)/meshes/right_wheel.stl" />
+      <mesh filename="package://racecar_description/meshes/right_wheel.stl" />
     </geometry>
   </xacro:macro>
@@ -53,5 +53,5 @@
     <origin xyz="0 0 0" rpy="0 0 0" />
     <geometry>
-      <mesh filename="file://$(find racecar_description)/meshes/left_wheel.stl" />
+      <mesh filename="package://racecar_description/meshes/left_wheel.stl" />
     </geometry>
   </xacro:macro>
@@ -59,5 +59,5 @@
     <origin xyz="0 0 0" rpy="0 0 0" />
     <geometry>
-      <mesh filename="file://$(find racecar_description)/meshes/right_wheel.stl" />
+      <mesh filename="package://racecar_description/meshes/right_wheel.stl" />
     </geometry>
   </xacro:macro>
@@ -65,5 +65,5 @@
     <origin xyz="0 0 0" rpy="0 0 0" />
     <geometry>
-      <mesh filename="file://$(find racecar_description)/meshes/hinge.stl" />
+      <mesh filename="package://racecar_description/meshes/hinge.stl" />
     </geometry>
   </xacro:macro>
@@ -71,5 +71,5 @@
     <origin xyz="0 0 0" rpy="0 0 0" />
     <geometry>
-      <mesh filename="file://$(find racecar_description)/meshes/hinge.stl" />
+      <mesh filename="package://racecar_description/meshes/hinge.stl" />
     </geometry>
   </xacro:macro>
@@ -268,5 +268,5 @@
       <origin xyz="0 0 0" rpy="0 0 0"/>
       <geometry>
-        <mesh filename="file://$(find racecar_description)/meshes/hokuyo.stl"/>
+        <mesh filename="package://racecar_description/meshes/hokuyo.stl"/>
         <material name="grey" />
       </geometry>
@@ -319,5 +319,5 @@
     <axis xyz="0 0 1" />
   </joint>
-  <ros2_control name="GazeboSystem" type="system">
+  <!-- <ros2_control name="GazeboSystem" type="system">
     <hardware>
       <plugin>gazebo_ros2_control/GazeboSystem</plugin>
@@ -331,4 +331,22 @@
       <state_interface name="velocity"/>
       <state_interface name="effort"/>
+    </joint>
+  </ros2_control> -->
+  <ros2_control name="VescVelocityInterface" type="system">
+    <hardware>
+      <plugin>racecar_hardware/VescInterface</plugin>
+      <param name="vesc_port">/dev/sensors/vesc</param>
+      <param name="erpm_gain">4614.0</param>
+      <param name="erpm_offset">0.0</param>
+      <param name="servo_gain">-1.2135</param>
+      <param name="servo_offset">0.5304</param>
+    </hardware>
+    <joint name="engine">
+      <command_interface name="velocity" />
+      <state_interface name="velocity" />
+    </joint>
+    <joint name="servo">
+      <command_interface name="position" />
+      <state_interface name="position"/>
     </joint>
   </ros2_control>
