Commit message: split up xacro files

File: src/racecar_description/urdf/racecar.urdf.xacro (robot description, xacro)
@@ -1,473 +1,5 @@
 <?xml version="1.0"?>
-<robot name="racecar"
-  xmlns:xacro="http://www.ros.org/wiki/xacro">
-  <!-- Global namespace -->
-  <xacro:arg name="robot_name" default="" />
-  <xacro:arg name="robot_skin" default="Blue" />
-  <!-- inertial parameter macros -->
-  <xacro:macro name="chassis_inertial_params">
-    <origin xyz="0.1477 0 0" rpy="0 0 0" />
-    <mass value="4.0" />
-    <inertia ixx="0.010609" ixy="0" ixz="0" iyy="0.050409" iyz="0" izz="0.05865" />
-  </xacro:macro>
-  <xacro:macro name="left_wheels_inertial_params">
-    <origin xyz="0 0 -0.0225" rpy="0 0 0" />
-    <mass value="0.34055" />
-    <inertia ixx="0.00026046" ixy="0" ixz="0" iyy="0.00026046" iyz="0" izz="0.00041226" />
-  </xacro:macro>
-  <xacro:macro name="right_wheels_inertial_params">
-    <origin xyz="0 0 0.0225" rpy="0 0 0" />
-    <mass value="0.34055" />
-    <inertia ixx="0.00026046" ixy="0" ixz="0" iyy="0.00026046" iyz="0" izz="0.00041226" />
-  </xacro:macro>
-  <xacro:macro name="steering_hinge_inertial_params">
-    <origin xyz="0 0 0" rpy="0 0 0" />
-    <mass value="0.100" />
-    <inertia ixx="4E-06" ixy="0" ixz="0" iyy="4E-06" iyz="0" izz="4E-06" />
-  </xacro:macro>
-  <xacro:macro name="hokuyo_inertial_params">
-    <origin xyz="0 0 0" rpy="0 0 0" />
-    <mass value="0.130" />
-    <inertia ixx="4E-06" ixy="0" ixz="0" iyy="4E-06" iyz="0" izz="4E-06" />
-  </xacro:macro>
-  <!-- geometry macros -->
-  <xacro:macro name="chassis_geometry">
-    <origin xyz="0.46 -0.135 -0.180" rpy="1.57 0 3.14" />
-    <geometry>
-      <mesh filename="package://racecar_description/meshes/chassis.stl" scale="0.000990 0.0009375 0.0009375"/>
-    </geometry>
-  </xacro:macro>
-  <xacro:macro name="left_rear_wheel_geometry">
-    <origin xyz="0 0 0" rpy="0 0 0" />
-    <geometry>
-      <mesh filename="package://racecar_description/meshes/left_wheel.stl" />
-    </geometry>
-  </xacro:macro>
-  <xacro:macro name="right_rear_wheel_geometry">
-    <origin xyz="0 0 0" rpy="0 0 0" />
-    <geometry>
-      <mesh filename="package://racecar_description/meshes/right_wheel.stl" />
-    </geometry>
-  </xacro:macro>
-  <xacro:macro name="left_front_wheel_geometry">
-    <origin xyz="0 0 0" rpy="0 0 0" />
-    <geometry>
-      <mesh filename="package://racecar_description/meshes/left_wheel.stl" />
-    </geometry>
-  </xacro:macro>
-  <xacro:macro name="right_front_wheel_geometry">
-    <origin xyz="0 0 0" rpy="0 0 0" />
-    <geometry>
-      <mesh filename="package://racecar_description/meshes/right_wheel.stl" />
-    </geometry>
-  </xacro:macro>
-  <xacro:macro name="left_steering_hinge_geometry">
-    <origin xyz="0 0 0" rpy="0 0 0" />
-    <geometry>
-      <mesh filename="package://racecar_description/meshes/hinge.stl" />
-    </geometry>
-  </xacro:macro>
-  <xacro:macro name="right_steering_hinge_geometry">
-    <origin xyz="0 0 0" rpy="0 0 0" />
-    <geometry>
-      <mesh filename="package://racecar_description/meshes/hinge.stl" />
-    </geometry>
-  </xacro:macro>
-  <xacro:macro name="left_wheels_collision_geometry">
-    <origin xyz="0 0 -0.0225" rpy="0 0 0" />
-    <geometry>
-      <cylinder length="0.045" radius="0.05" />
-    </geometry>
-  </xacro:macro>
-  <xacro:macro name="right_wheels_collision_geometry">
-    <origin xyz="0 0 0.0225" rpy="0 0 0" />
-    <geometry>
-      <cylinder length="0.045" radius="0.05" />
-    </geometry>
-  </xacro:macro>
-  <!-- transmission macros -->
-  <xacro:macro name="wheel_transmission" params="name">
-    <transmission name="${name}_transmission" type="SimpleTransmission">
-      <type>transmission_interface/SimpleTransmission</type>
-      <joint name="${name}_joint">
-        <hardwareInterface>hardware_interface/EffortJointInterface</hardwareInterface>
-      </joint>
-      <actuator name="${name}_motor">
-        <hardwareInterface>hardware_interface/EffortJointInterface</hardwareInterface>
-        <mechanicalReduction>1</mechanicalReduction>
-      </actuator>
-    </transmission>
-  </xacro:macro>
-  <xacro:macro name="steering_hinge_transmission" params="name">
-    <transmission name="${name}_transmission" type="SimpleTransmission">
-      <type>transmission_interface/SimpleTransmission</type>
-      <joint name="${name}_joint">
-        <hardwareInterface>hardware_interface/EffortJointInterface</hardwareInterface>
-      </joint>
-      <actuator name="${name}_motor">
-        <hardwareInterface>hardware_interface/EffortJointInterface</hardwareInterface>
-        <mechanicalReduction>1</mechanicalReduction>
-      </actuator>
-    </transmission>
-  </xacro:macro>
-  <!-- Add chassis and it's inertia link -->
-  <link name="$(arg robot_name)base_link"/>
-  <link name="$(arg robot_name)chassis">
-    <visual>
-      <xacro:chassis_geometry/>
-      <material name="red" />
-    </visual>
-  </link>
-  <joint name="$(arg robot_name)base_link_joint" type="fixed">
-    <origin xyz="0 0 0.05" rpy="0 0 0" />
-    <parent link="$(arg robot_name)base_link" />
-    <child link="$(arg robot_name)chassis" />
-  </joint>
-  <link name="$(arg robot_name)chassis_inertia">
-    <inertial>
-      <xacro:chassis_inertial_params />
-    </inertial>
-  </link>
-  <joint name="$(arg robot_name)chassis_inertia_joint" type="fixed">
-    <origin xyz="0 0 0" rpy="0 0 0" />
-    <parent link="$(arg robot_name)chassis" />
-    <child link="$(arg robot_name)chassis_inertia" />
-  </joint>
-  <!-- Add the left rear wheel with its joints and tranmissions -->
-  <link name="$(arg robot_name)left_rear_wheel">
-    <inertial>
-      <xacro:left_wheels_inertial_params />
-    </inertial>
-    <visual>
-      <xacro:left_rear_wheel_geometry />
-      <material name="black" />
-    </visual>
-    <collision>
-      <xacro:left_wheels_collision_geometry />
-    </collision>
-  </link>
-  <joint name="$(arg robot_name)left_rear_wheel_joint" type="continuous">
-    <origin xyz="0 0.1 0" rpy="1.5708 0 0" />
-    <parent link="$(arg robot_name)chassis" />
-    <child link="$(arg robot_name)left_rear_wheel" />
-    <axis xyz="0 0 -1" />
-    <limit effort="10" velocity="100" />
-  </joint>
-  <xacro:wheel_transmission name="$(arg robot_name)left_rear_wheel" />
-  <!-- Add the right rear wheel with its joints and tranmissions -->
-  <link name="$(arg robot_name)right_rear_wheel">
-    <inertial>
-      <xacro:right_wheels_inertial_params />
-    </inertial>
-    <visual>
-      <xacro:right_rear_wheel_geometry />
-      <material name="black" />
-    </visual>
-    <collision>
-      <xacro:right_wheels_collision_geometry />
-    </collision>
-  </link>
-  <joint name="$(arg robot_name)right_rear_wheel_joint" type="continuous">
-    <origin xyz="0 -0.1 0" rpy="1.5708 0 0" />
-    <parent link="$(arg robot_name)chassis" />
-    <child link="$(arg robot_name)right_rear_wheel" />
-    <axis xyz="0 0 -1" />
-    <limit effort="10" velocity="100" />
-  </joint>
-  <xacro:wheel_transmission name="$(arg robot_name)right_rear_wheel" />
-  <!-- Add the left steering hinge with its joints and tranmissions -->
-  <link name="$(arg robot_name)left_steering_hinge">
-    <inertial>
-      <xacro:steering_hinge_inertial_params />
-    </inertial>
-    <visual>
-      <xacro:left_steering_hinge_geometry />
-      <material name="grey" />
-    </visual>
-  </link>
-  <joint name="$(arg robot_name)left_steering_hinge_joint" type="revolute">
-    <origin xyz="0.325 0.1 0" rpy="0 1.5708 0" />
-    <parent link="$(arg robot_name)chassis" />
-    <child link="$(arg robot_name)left_steering_hinge" />
-    <axis xyz="-1 0 0" />
-    <limit lower="-1.0" upper="1.0" effort="10" velocity="100" />
-  </joint>
-  <xacro:steering_hinge_transmission name="$(arg robot_name)left_steering_hinge" />
-  <!-- Add the right steering hinge with its joints and tranmissions -->
-  <link name="$(arg robot_name)right_steering_hinge">
-    <inertial>
-      <xacro:steering_hinge_inertial_params />
-    </inertial>
-    <visual>
-      <xacro:right_steering_hinge_geometry />
-      <material name="grey" />
-    </visual>
-  </link>
-  <joint name="$(arg robot_name)right_steering_hinge_joint" type="revolute">
-    <origin xyz="0.325 -0.1 0" rpy="0 1.5708 0" />
-    <parent link="$(arg robot_name)chassis" />
-    <child link="$(arg robot_name)right_steering_hinge" />
-    <axis xyz="-1 0 0" />
-    <limit lower="-1.0" upper="1.0" effort="10" velocity="100" />
-  </joint>
-  <xacro:steering_hinge_transmission name="$(arg robot_name)right_steering_hinge" />
-  <!-- Add the left front wheel with its joints and tranmissions -->
-  <link name="$(arg robot_name)left_front_wheel">
-    <inertial>
-      <xacro:left_wheels_inertial_params />
-    </inertial>
-    <visual>
-      <xacro:left_front_wheel_geometry />
-      <material name="black" />
-    </visual>
-    <collision>
-      <xacro:left_wheels_collision_geometry />
-    </collision>
-  </link>
-  <joint name="$(arg robot_name)left_front_wheel_joint" type="continuous">
-    <origin xyz="0 0 0" rpy="1.5708 0 0" />
-    <parent link="$(arg robot_name)left_steering_hinge" />
-    <child link="$(arg robot_name)left_front_wheel" />
-    <axis xyz="0 0 -1" />
-    <limit effort="10" velocity="100" />
-  </joint>
-  <xacro:wheel_transmission name="$(arg robot_name)left_front_wheel" />
-  <!-- Add the left front wheel with its joints and tranmissions -->
-  <link name="$(arg robot_name)right_front_wheel">
-    <inertial>
-      <xacro:right_wheels_inertial_params />
-    </inertial>
-    <visual>
-      <xacro:right_front_wheel_geometry />
-      <material name="black" />
-    </visual>
-    <collision>
-      <xacro:right_wheels_collision_geometry />
-    </collision>
-  </link>
-  <joint name="$(arg robot_name)right_front_wheel_joint" type="continuous">
-    <origin xyz="0 0 0" rpy="1.5708 0 0" />
-    <parent link="$(arg robot_name)right_steering_hinge" />
-    <child link="$(arg robot_name)right_front_wheel" />
-    <axis xyz="0 0 -1" />
-    <limit effort="10" velocity="100"/>
-  </joint>
-  <xacro:wheel_transmission name="$(arg robot_name)right_front_wheel" />
-  <!-- Add Hokuyo laser scanner -->
-  <link name="$(arg robot_name)laser_link">
-    <inertial>
-      <xacro:hokuyo_inertial_params />
-    </inertial>
-    <collision>
-      <origin xyz="0 0 0" rpy="0 0 0"/>
-      <geometry>
-        <box size="0.1 0.1 0.1"/>
-      </geometry>
-    </collision>
-    <visual>
-      <origin xyz="0 0 0" rpy="0 0 0"/>
-      <geometry>
-        <mesh filename="package://racecar_description/meshes/hokuyo.stl"/>
-        <material name="grey" />
-      </geometry>
-    </visual>
-  </link>
-  <joint name="$(arg robot_name)hokuyo_joint" type="fixed">
-    <origin xyz="0.125 0.0 0.155" rpy="0 0 0"/>
-    <parent link="$(arg robot_name)chassis" />
-    <child link="$(arg robot_name)laser_link" />
-    <axis xyz="0 0 1" />
-  </joint>
-  <link name="$(arg robot_name)link">
-    <inertial>
-      <mass value="1e-5" />
-      <origin xyz="0 0 0.25" rpy="0 0 0"/>
-      <inertia ixx="1e-6" ixy="0" ixz="0" iyy="1e-6" iyz="0" izz="1e-6" />
-    </inertial>
-    <collision>
-      <origin xyz="0 0 0.25" rpy="0 0 0"/>
-      <geometry>
-        <box size="0.033 0.175 0.030"/>
-      </geometry>
-    </collision>
-    <visual>
-      <origin xyz="0 0 0.025" rpy="0 0 0"/>
-      <geometry>
-        <box size="0.033 0.175 0.030"/>
-      </geometry>
-      <material name="red"/>
-    </visual>
-  </link>
-  <joint name="$(arg robot_name)joint" type="fixed">
-    <origin xyz="0.390 0 0.025" rpy="0 0 0"/>
-    <parent link="$(arg robot_name)chassis"/>
-    <child link="$(arg robot_name)link"/>
-    <axis xyz="0 0 1" />
-    <!-- <limit lower="0.0" upper="0.0" effort="0.0" velocity="0.0" /> -->
-  </joint>
-  <link name="$(arg robot_name)right_link">
-    <inertial>
-      <mass value="1e-5" />
-      <origin xyz="-2.5 0 1.75" rpy="0 .57 0"/>
-      <inertia ixx="1e-6" ixy="0" ixz="0" iyy="1e-6" iyz="0" izz="1e-6" />
-    </inertial>
-  </link>
-  <joint name="$(arg robot_name)right_joint" type="fixed">
-    <origin xyz="0 -0.06 0.025" rpy="0 0 0"/>
-    <parent link="$(arg robot_name)link"/>
-    <child link="$(arg robot_name)right_link"/>
-    <axis xyz="0 0 1" />
-  </joint>
-  <!-- <ros2_control name="GazeboSystem" type="system">
-    <hardware>
-      <plugin>gazebo_ros2_control/GazeboSystem</plugin>
-    </hardware>
-    <joint name="slider_to_cart">
-      <command_interface name="effort">
-        <param name="min">-1000</param>
-        <param name="max">1000</param>
-      </command_interface>
-      <state_interface name="position"/>
-      <state_interface name="velocity"/>
-      <state_interface name="effort"/>
-    </joint>
-  </ros2_control> -->
-  <ros2_control name="VescVelocityInterface" type="system">
-    <hardware>
-      <plugin>racecar_hardware/VescInterface</plugin>
-      <param name="vesc_port">/dev/sensors/vesc</param>
-      <param name="erpm_gain">4614.0</param>
-      <param name="erpm_offset">0.0</param>
-      <param name="servo_gain">-1.2135</param>
-      <param name="servo_offset">0.5304</param>
-    </hardware>
-    <joint name="engine">
-      <command_interface name="velocity" />
-      <state_interface name="velocity" />
-    </joint>
-    <joint name="servo">
-      <command_interface name="position" />
-      <state_interface name="position"/>
-    </joint>
-  </ros2_control>
-  <!-- Gazebo references -->
-  <gazebo reference="$(arg robot_name)chassis">
-    <mu1 value="0.0"/>
-    <mu2 value="0.0"/>
-    <kp value="10000000.0" />
-    <kd value="1.0" />
-    <material>Gazebo/$(arg robot_skin)</material>
-  </gazebo>
-  <gazebo reference="$(arg robot_name)left_rear_wheel">
-    <mu1 value="1.0"/>
-    <mu2 value="1.0"/>
-    <kp value="10000000.0" />
-    <kd value="1.0" />
-    <fdir1 value="1 0 0"/>
-    <material>Gazebo/Black</material>
-  </gazebo>
-  <gazebo reference="$(arg robot_name)right_rear_wheel">
-    <mu1 value="1.0"/>
-    <mu2 value="1.0"/>
-    <kp value="10000000.0" />
-    <kd value="1.0" />
-    <fdir1 value="1 0 0"/>
-    <material>Gazebo/Black</material>
-  </gazebo>
-  <gazebo reference="$(arg robot_name)left_front_wheel">
-    <mu1 value="1.0"/>
-    <mu2 value="1.0"/>
-    <kp value="10000000.0" />
-    <kd value="1.0" />
-    <fdir1 value="0 0 1"/>
-    <material>Gazebo/Black</material>
-  </gazebo>
-  <gazebo reference="$(arg robot_name)right_front_wheel">
-    <mu1 value="1.0"/>
-    <mu2 value="1.0"/>
-    <kp value="10000000.0" />
-    <kd value="1.0" />
-    <fdir1 value="0 0 1"/>
-    <material>Gazebo/Black</material>
-  </gazebo>
-  <!-- Gazebo plugins
-  <gazebo>
-    <plugin name="gazebo_ros_control" filename="libgazebo_ros_control.so">
-      <robotNamespace>/$(arg robot_name)</robotNamespace>
-      <robotSimType>gazebo_ros_control/DefaultRobotHWSim</robotSimType>
-    </plugin>
-  </gazebo>
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