Commit message: renamed joint

File: src/racecar_description/urdf/hardware_interfaces/vesc.xacro (robot description, xacro)
@@ -13,5 +13,5 @@
             <param name="use_current">1</param>
         </hardware>
-        <joint name="drive_train">
+        <joint name="motor">
             <command_interface name="duty_cycle">
                 <param name="min">0.05</param>

File: src/racecar_description/urdf/racecar.urdf.xacro (robot description, xacro)
@@ -2,5 +2,5 @@
 <robot name="racecar" xmlns:xacro="http://www.ros.org/wiki/xacro">
   <xacro:include filename="$(find racecar_description)/urdf/description.urdf.xacro" />
-  <xacro:include filename="$(find racecar_description)/urdf/control_interfaces/vesc.xacro" />
+  <xacro:include filename="$(find racecar_description)/urdf/hardware_interfaces/vesc.xacro" />
   <!-- <xacro:include filename="$(find racecar_description)/urdf/control_interfaces/velocity.xacro" />-->
 </robot>
